File: MCP2551_STM32_tryout.kicad_sch (KiCad schematic)
At the start: 0 parts

Commit message: update,
Parts:
- added C? (x2): C561,0805, Capacitor_SMD:C_0805_2012Metric_Pad1.15x1.40mm_HandSolder, symbol taobao-c:C561,0805
- added C?: C104, symbol taobao-c:C104
- added D?: PESD1CAN, symbol taobao-components:PESD1CAN
- added J?: Conn_01x02, symbol Connector_Generic:Conn_01x02
- added R?: R121,0805, Resistor_SMD:R_0805_2012Metric_Pad1.15x1.40mm_HandSolder, symbol taobao-r:R121,0805
- added R? (x2): R101,0805, Resistor_SMD:R_0805_2012Metric_Pad1.15x1.40mm_HandSolder, symbol taobao-r:R101,0805
- added R?: R472,0805, Resistor_SMD:R_0805_2012Metric_Pad1.15x1.40mm_HandSolder, symbol taobao-r:R472,0805
- added U?: MCP2551, Package_SO:SOIC-8_3.9x4.9mm_P1.27mm, symbol taobao-components:MCP2551
Connections:
- new net: C?.1, R?.2 (x2)
- new net: R?.2, U?.8 (Rs)
- new net +5V: C?.1, U?.3 (VDD)
- new net CANH: D?.1, J?.1 (Pin_1), R?.1, R?.1, U?.7 (CANH)
- new net CANL: D?.2, J?.2 (Pin_2), R?.1, R?.2, U?.6 (CANL)
- new net CAN_RXD: U?.4 (RXD)
- new net CAN_TXD: U?.1 (TXD)
- new net GND: C?.2, C?.2, C?.2, D?.3, R?.1, U?.2 (VSS)

Commit message: update,
Parts:
- removed C? (x2): C561,0805, Capacitor_SMD:C_0805_2012Metric_Pad1.15x1.40mm_HandSolder, symbol taobao-c:C561,0805
- removed C?: C104, symbol taobao-c:C104
- removed D?: PESD1CAN, symbol taobao-components:PESD1CAN
- removed J?: Conn_01x02, symbol Connector_Generic:Conn_01x02
- removed R?: R121,0805, Resistor_SMD:R_0805_2012Metric_Pad1.15x1.40mm_HandSolder, symbol taobao-r:R121,0805
- removed R? (x2): R101,0805, Resistor_SMD:R_0805_2012Metric_Pad1.15x1.40mm_HandSolder, symbol taobao-r:R101,0805
- removed R?: R472,0805, Resistor_SMD:R_0805_2012Metric_Pad1.15x1.40mm_HandSolder, symbol taobao-r:R472,0805
- removed U?: MCP2551, Package_SO:SOIC-8_3.9x4.9mm_P1.27mm, symbol taobao-components:MCP2551
Other:
- added sheet stm32_1 (stm32_1.kicad_sch)
- added sheet stm32_2 (stm32_2.kicad_sch)
- added sheet stm32_3 (stm32_3.kicad_sch)
