File: stm32_3.kicad_sch (KiCad schematic)
At the start: 11 parts, among them J3 Conn_01x02, U5 YAAJ_BluePill_Part_Like_SWD_B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, U6 MCP2551

Commit message: update,
Parts:
- added JP? (x2): SolderJumper_2_Open_arrow, Jumper:SolderJumper-2_P1.3mm_Open_TrianglePad1.0x1.5mm, symbol my_solder_jumper:SolderJumper_2_Open_arrow
Connections:
- net CAN_H: now also JP?.2 (B); no longer D3.1, J3.1 (Pin_1), R11.1, R12.1, U6.7 (CANH)
- net CAN_L: now also JP?.2 (B); no longer D3.2, J3.2 (Pin_2), R10.1, R12.2, U6.6 (CANL)
- new net CANH: D3.1, J3.1 (Pin_1), JP?.1 (A), R11.1, R12.1, U6.7 (CANH)
- new net CANL: D3.2, J3.2 (Pin_2), JP?.1 (A), R10.1, R12.2, U6.6 (CANL)
Changed lines of the file:
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@@
 (kicad_sch (version 20211123) (generator eeschema)
   (paper "A4")
-  (junction (at 236.22 73.66) (diameter 0) (color 0 0 0 0)
-  )
   (junction (at 215.9 73.66) (diameter 0) (color 0 0 0 0)
   )
@@
   (junction (at 180.34 86.36) (diameter 0) (color 0 0 0 0)
   )
+  (junction (at 233.68 73.66) (diameter 0) (color 0 0 0 0)
+  )
   (junction (at 208.28 86.36) (diameter 0) (color 0 0 0 0)
   )
   (junction (at 215.9 83.82) (diameter 0) (color 0 0 0 0)
   )
-  (junction (at 246.38 76.2) (diameter 0) (color 0 0 0 0)
+  (junction (at 243.84 76.2) (diameter 0) (color 0 0 0 0)
   )
   (wire (pts (xy 104.14 78.74) (xy 104.14 83.82))
@@
     (stroke (width 0) (type default) (color 0 0 0 0))
   )
-  (wire (pts (xy 236.22 68.58) (xy 236.22 73.66))
-    (stroke (width 0) (type default) (color 0 0 0 0))
-  )
   (wire (pts (xy 165.1 93.98) (xy 165.1 88.9))
     (stroke (width 0) (type default) (color 0 0 0 0))
@@
     (stroke (width 0) (type default) (color 0 0 0 0))
   )
+  (wire (pts (xy 243.84 76.2) (xy 261.62 76.2))
+    (stroke (width 0) (type default) (color 0 0 0 0))
+  )
   (wire (pts (xy 20.32 119.38) (xy 20.32 124.46))
     (stroke (width 0) (type default) (color 0 0 0 0))
@@
     (stroke (width 0) (type default) (color 0 0 0 0))
   )
-  (wire (pts (xy 236.22 73.66) (xy 261.62 73.66))
-    (stroke (width 0) (type default) (color 0 0 0 0))
-  )
   (wire (pts (xy 160.02 86.36) (xy 170.18 86.36))
     (stroke (width 0) (type default) (color 0 0 0 0))
@@
     (stroke (width 0) (type default) (color 0 0 0 0))
   )
-  (wire (pts (xy 246.38 76.2) (xy 261.62 76.2))
-    (stroke (width 0) (type default) (color 0 0 0 0))
-  )
   (wire (pts (xy 180.34 99.06) (xy 180.34 106.68))
     (stroke (width 0) (type default) (color 0 0 0 0))
@@
     (stroke (width 0) (type default) (color 0 0 0 0))
   )
-  (wire (pts (xy 233.68 76.2) (xy 246.38 76.2))
+  (wire (pts (xy 233.68 76.2) (xy 243.84 76.2))
+    (stroke (width 0) (type default) (color 0 0 0 0))
+  )
+  (wire (pts (xy 233.68 50.8) (xy 233.68 73.66))
     (stroke (width 0) (type default) (color 0 0 0 0))
   )
@@
     (stroke (width 0) (type default) (color 0 0 0 0))
   )
+  (wire (pts (xy 255.27 55.88) (xy 259.08 55.88))
+    (stroke (width 0) (type default) (color 0 0 0 0))
+  )
   (wire (pts (xy 195.58 73.66) (xy 195.58 93.98))
     (stroke (width 0) (type default) (color 0 0 0 0))
   )
+  (wire (pts (xy 247.65 50.8) (xy 233.68 50.8))
+    (stroke (width 0) (type default) (color 0 0 0 0))
+  )
   (wire (pts (xy 172.72 83.82) (xy 172.72 86.36))
     (stroke (width 0) (type default) (color 0 0 0 0))
@@
     (stroke (width 0) (type default) (color 0 0 0 0))
   )
-  (wire (pts (xy 246.38 68.58) (xy 246.38 76.2))
-    (stroke (width 0) (type default) (color 0 0 0 0))
-  )
-  (wire (pts (xy 215.9 73.66) (xy 236.22 73.66))
+  (wire (pts (xy 215.9 73.66) (xy 233.68 73.66))
     (stroke (width 0) (type default) (color 0 0 0 0))
   )
@@
     (stroke (width 0) (type default) (color 0 0 0 0))
   )
+  (wire (pts (xy 243.84 55.88) (xy 243.84 76.2))
+    (stroke (width 0) (type default) (color 0 0 0 0))
+  )
   (wire (pts (xy 104.14 83.82) (xy 134.62 83.82))
     (stroke (width 0) (type default) (color 0 0 0 0))
@@
     (stroke (width 0) (type default) (color 0 0 0 0))
   )
+  (wire (pts (xy 247.65 55.88) (xy 243.84 55.88))
+    (stroke (width 0) (type default) (color 0 0 0 0))
+  )
+  (wire (pts (xy 233.68 73.66) (xy 261.62 73.66))
+    (stroke (width 0) (type default) (color 0 0 0 0))
+  )
   (wire (pts (xy 195.58 114.3) (xy 195.58 111.76))
     (stroke (width 0) (type default) (color 0 0 0 0))
@@
   )
   (wire (pts (xy 210.82 73.66) (xy 215.9 73.66))
+    (stroke (width 0) (type default) (color 0 0 0 0))
+  )
+  (wire (pts (xy 255.27 50.8) (xy 259.08 50.8))
     (stroke (width 0) (type default) (color 0 0 0 0))
   )
@@
     (effects (font (size 1.27 1.27)) (justify right bottom))
   )
-  (hierarchical_label "CAN_L" (shape bidirectional) (at 246.38 68.58 90)
+  (hierarchical_label "CAN_H" (shape bidirectional) (at 259.08 50.8 0)
     (effects (font (size 1.27 1.27)) (justify left))
   )
-  (hierarchical_label "CAN_H" (shape bidirectional) (at 236.22 68.58 90)
+  (hierarchical_label "CAN_L" (shape bidirectional) (at 259.08 55.88 0)
     (effects (font (size 1.27 1.27)) (justify left))
   )
@@
     (pin "1")
   )
+  (symbol (lib_id "my_solder_jumper:SolderJumper_2_Open_arrow") (at 251.46 55.88 0) (unit 1)
+    (in_bom yes) (on_board yes) (fields_autoplaced)
+    (property "Reference" "JP?" (id 0) (at 251.46 49.53 0))
+    (property "Value" "SolderJumper_2_Open_arrow" (id 1) (at 251.46 52.07 0))
+    (property "Footprint" "Jumper:SolderJumper-2_P1.3mm_Open_TrianglePad1.0x1.5mm" (id 2) (at 251.46 55.88 0)
+      (effects (font (size 1.27 1.27)) hide)
+    )
+    (property "Datasheet" "~" (id 3) (at 251.46 55.88 0)
+      (effects (font (size 1.27 1.27)) hide)
+    )
+    (pin "1")
+    (pin "2")
+  )
+  (symbol (lib_id "my_solder_jumper:SolderJumper_2_Open_arrow") (at 251.46 50.8 0) (unit 1)
+    (in_bom yes) (on_board yes) (fields_autoplaced)
+    (property "Reference" "JP?" (id 0) (at 251.46 44.45 0))
+    (property "Value" "SolderJumper_2_Open_arrow" (id 1) (at 251.46 46.99 0))
+    (property "Footprint" "Jumper:SolderJumper-2_P1.3mm_Open_TrianglePad1.0x1.5mm" (id 2) (at 251.46 50.8 0)
+      (effects (font (size 1.27 1.27)) hide)
+    )
+    (property "Datasheet" "~" (id 3) (at 251.46 50.8 0)
+      (effects (font (size 1.27 1.27)) hide)
+    )
+    (pin "1")
+    (pin "2")
+  )
   (symbol (lib_id "taobao-components:MCP2551") (at 147.32 83.82 0) (mirror x) (unit 1)

Commit message: update,
Parts:
- added H? (x4): MountingHole, footprint-lib:MountingHole_3.1mm_M3,rpi_like, symbol Mechanical:MountingHole
- gave numbers to parts that had none: 2
Changed lines of the file:
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@@
   (symbol (lib_id "power:+5V") (at 76.2 73.66 0) (unit 1)
     (in_bom yes) (on_board yes) (fields_autoplaced)
-    (property "Reference" "#PWR?" (id 0) (at 76.2 77.47 0)
+    (property "Reference" "#PWR0121" (id 0) (at 76.2 77.47 0)
       (effects (font (size 1.27 1.27)) hide)
     )
@@
     )
     (pin "1")
+  )
+  (symbol (lib_id "Mechanical:MountingHole") (at 149.86 187.96 0) (unit 1)
+    (in_bom yes) (on_board yes) (fields_autoplaced)
+    (property "Reference" "H?" (id 0) (at 152.4 186.6899 0)
+      (effects (font (size 1.27 1.27)) (justify left))
+    )
+    (property "Value" "MountingHole" (id 1) (at 152.4 189.2299 0)
+      (effects (font (size 1.27 1.27)) (justify left))
+    )
+    (property "Footprint" "footprint-lib:MountingHole_3.1mm_M3,rpi_like" (id 2) (at 149.86 187.96 0)
+      (effects (font (size 1.27 1.27)) hide)
+    )
+    (property "Datasheet" "~" (id 3) (at 149.86 187.96 0)
+      (effects (font (size 1.27 1.27)) hide)
+    )
   )
   (symbol (lib_id "taobao-c:C561,0805") (at 195.58 109.22 0) (unit 1)
@@
     (pin "1")
   )
+  (symbol (lib_id "Mechanical:MountingHole") (at 149.86 177.8 0) (unit 1)
+    (in_bom yes) (on_board yes) (fields_autoplaced)
+    (property "Reference" "H?" (id 0) (at 152.4 176.5299 0)
+      (effects (font (size 1.27 1.27)) (justify left))
+    )
+    (property "Value" "MountingHole" (id 1) (at 152.4 179.0699 0)
+      (effects (font (size 1.27 1.27)) (justify left))
+    )
+    (property "Footprint" "footprint-lib:MountingHole_3.1mm_M3,rpi_like" (id 2) (at 149.86 177.8 0)
+      (effects (font (size 1.27 1.27)) hide)
+    )
+    (property "Datasheet" "~" (id 3) (at 149.86 177.8 0)
+      (effects (font (size 1.27 1.27)) hide)
+    )
+  )
   (symbol (lib_id "my_solder_jumper:SolderJumper_2_Open_arrow") (at 251.46 55.88 0) (unit 1)
     (in_bom yes) (on_board yes) (fields_autoplaced)
-    (property "Reference" "JP?" (id 0) (at 251.46 49.53 0))
+    (property "Reference" "JP6" (id 0) (at 251.46 49.53 0))
     (property "Value" "SolderJumper_2_Open_arrow" (id 1) (at 251.46 52.07 0))
     (property "Footprint" "Jumper:SolderJumper-2_P1.3mm_Open_TrianglePad1.0x1.5mm" (id 2) (at 251.46 55.88 0)
@@
   (symbol (lib_id "my_solder_jumper:SolderJumper_2_Open_arrow") (at 251.46 50.8 0) (unit 1)
     (in_bom yes) (on_board yes) (fields_autoplaced)
-    (property "Reference" "JP?" (id 0) (at 251.46 44.45 0))
+    (property "Reference" "JP5" (id 0) (at 251.46 44.45 0))
     (property "Value" "SolderJumper_2_Open_arrow" (id 1) (at 251.46 46.99 0))
     (property "Footprint" "Jumper:SolderJumper-2_P1.3mm_Open_TrianglePad1.0x1.5mm" (id 2) (at 251.46 50.8 0)
@@
     (pin "8")
   )
+  (symbol (lib_id "Mechanical:MountingHole") (at 149.86 182.88 0) (unit 1)
+    (in_bom yes) (on_board yes) (fields_autoplaced)
+    (property "Reference" "H?" (id 0) (at 152.4 181.6099 0)
+      (effects (font (size 1.27 1.27)) (justify left))
+    )
+    (property "Value" "MountingHole" (id 1) (at 152.4 184.1499 0)
+      (effects (font (size 1.27 1.27)) (justify left))
+    )
+    (property "Footprint" "footprint-lib:MountingHole_3.1mm_M3,rpi_like" (id 2) (at 149.86 182.88 0)
+      (effects (font (size 1.27 1.27)) hide)
+    )
+    (property "Datasheet" "~" (id 3) (at 149.86 182.88 0)
+      (effects (font (size 1.27 1.27)) hide)
+    )
+  )
   (symbol (lib_id "power:GND") (at 104.14 99.06 0) (unit 1)
     (in_bom yes) (on_board yes) (fields_autoplaced)
@@
     (pin "1")
     (pin "2")
+  )
+  (symbol (lib_id "Mechanical:MountingHole") (at 149.86 172.72 0) (unit 1)
+    (in_bom yes) (on_board yes) (fields_autoplaced)
+    (property "Reference" "H?" (id 0) (at 152.4 171.4499 0)
+      (effects (font (size 1.27 1.27)) (justify left))
+    )
+    (property "Value" "MountingHole" (id 1) (at 152.4 173.9899 0)
+      (effects (font (size 1.27 1.27)) (justify left))
+    )
+    (property "Footprint" "footprint-lib:MountingHole_3.1mm_M3,rpi_like" (id 2) (at 149.86 172.72 0)
+      (effects (font (size 1.27 1.27)) hide)
+    )
+    (property "Datasheet" "~" (id 3) (at 149.86 172.72 0)
+      (effects (font (size 1.27 1.27)) hide)
+    )
   )
   (symbol (lib_id "taobao-r:R121,0805") (at 215.9 78.74 0) (unit 1)
@@
   (symbol (lib_id "power:GND") (at 20.32 124.46 0) (unit 1)
     (in_bom yes) (on_board yes) (fields_autoplaced)
-    (property "Reference" "#PWR?" (id 0) (at 20.32 130.81 0)
-      (effects (font (size 1.27 1.27)) hide)
-    )
+    (property "Reference" "#PWR0120" (id 0) (at 20.32 130.81 0)
+      (effects (font (size 1.27 1.27)) hide)
+    )

Commit message: update,
Parts:
- removed H? (x2): MountingHole, footprint-lib:MountingHole_3.1mm_M3,rpi_like, symbol Mechanical:MountingHole
- H? (x2): footprint footprint-lib:MountingHole_3.1mm_M3,rpi_like -> (none)
Changed lines of the file:
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@@
     (pin "1")
-  )
-  (symbol (lib_id "Mechanical:MountingHole") (at 149.86 187.96 0) (unit 1)
-    (in_bom yes) (on_board yes) (fields_autoplaced)
-    (property "Reference" "H?" (id 0) (at 152.4 186.6899 0)
-      (effects (font (size 1.27 1.27)) (justify left))
-    )
-    (property "Value" "MountingHole" (id 1) (at 152.4 189.2299 0)
-      (effects (font (size 1.27 1.27)) (justify left))
-    )
-    (property "Footprint" "footprint-lib:MountingHole_3.1mm_M3,rpi_like" (id 2) (at 149.86 187.96 0)
-      (effects (font (size 1.27 1.27)) hide)
-    )
-    (property "Datasheet" "~" (id 3) (at 149.86 187.96 0)
-      (effects (font (size 1.27 1.27)) hide)
-    )
   )
   (symbol (lib_id "taobao-c:C561,0805") (at 195.58 109.22 0) (unit 1)
@@
       (effects (font (size 1.27 1.27)) (justify left))
     )
-    (property "Footprint" "footprint-lib:MountingHole_3.1mm_M3,rpi_like" (id 2) (at 149.86 177.8 0)
+    (property "Footprint" "" (id 2) (at 149.86 177.8 0)
       (effects (font (size 1.27 1.27)) hide)
     )
@@
     (pin "8")
   )
-  (symbol (lib_id "Mechanical:MountingHole") (at 149.86 182.88 0) (unit 1)
-    (in_bom yes) (on_board yes) (fields_autoplaced)
-    (property "Reference" "H?" (id 0) (at 152.4 181.6099 0)
-      (effects (font (size 1.27 1.27)) (justify left))
-    )
-    (property "Value" "MountingHole" (id 1) (at 152.4 184.1499 0)
-      (effects (font (size 1.27 1.27)) (justify left))
-    )
-    (property "Footprint" "footprint-lib:MountingHole_3.1mm_M3,rpi_like" (id 2) (at 149.86 182.88 0)
-      (effects (font (size 1.27 1.27)) hide)
-    )
-    (property "Datasheet" "~" (id 3) (at 149.86 182.88 0)
-      (effects (font (size 1.27 1.27)) hide)
-    )
-  )
   (symbol (lib_id "power:GND") (at 104.14 99.06 0) (unit 1)
     (in_bom yes) (on_board yes) (fields_autoplaced)
@@
       (effects (font (size 1.27 1.27)) (justify left))
     )
-    (property "Footprint" "footprint-lib:MountingHole_3.1mm_M3,rpi_like" (id 2) (at 149.86 172.72 0)
-      (effects (font (size 1.27 1.27)) hide)
-    )
+    (property "Footprint" "" (id 2) (at 149.86 172.72 0)
+      (effects (font (size 1.27 1.27)) hide)
+    )
