File: MCP2551_STM32_tryout.kicad_pcb (KiCad board)
At the start: 2 copper layers, 95 x 95 mm, 15 parts, among them J1 Conn_01x02, J2 Conn_01x02, J3 Conn_01x02, U1 YAAJ_BluePill_Part_Like_SWD_B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, U2 MCP2551, U3 YAAJ_BluePill_Part_Like_SWD_B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, U4 MCP2551, U5 YAAJ_BluePill_Part_Like_SWD_B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, U6 MCP2551

Commit message: update,
Parts:
- added C2: C561,0805, Capacitor_SMD:C_0805_2012Metric, F.Cu at (70.0, 37.5)
- added C3: C561,0805, Capacitor_SMD:C_0805_2012Metric, F.Cu at (74.5, 37.5)
- added C5: C561,0805, Capacitor_SMD:C_0805_2012Metric, F.Cu at (82.9, 28.9)
- added C6: C561,0805, Capacitor_SMD:C_0805_2012Metric, F.Cu at (87.4, 28.9)
- added C8: C561,0805, Capacitor_SMD:C_0805_2012Metric, F.Cu at (-37.4, 19.7)
- added C9: C561,0805, Capacitor_SMD:C_0805_2012Metric, F.Cu at (-30.5, 19.8)
- added R1: R472,0805, Resistor_SMD:R_0805_2012Metric, F.Cu at (95.0, 45.0)
- added R10: R101,0805, Resistor_SMD:R_0805_2012Metric, F.Cu at (-34.9, 19.7)
- added R11: R101,0805, Resistor_SMD:R_0805_2012Metric, F.Cu at (-27.9, 19.8)
- added R12: R121,0805, Resistor_SMD:R_0805_2012Metric, F.Cu at (-30.5, 38.1)
- added R2: R101,0805, Resistor_SMD:R_0805_2012Metric, F.Cu at (90.6, 45.0)
- added R3: R101,0805, Resistor_SMD:R_0805_2012Metric, F.Cu at (95.0, 48.0)
- added R4: R121,0805, Resistor_SMD:R_0805_2012Metric, F.Cu at (90.6, 48.0)
- added R5: R472,0805, Resistor_SMD:R_0805_2012Metric, F.Cu at (105.1, 38.5)
- added R6: R101,0805, Resistor_SMD:R_0805_2012Metric, F.Cu at (105.1, 35.5)
- added R7: R101,0805, Resistor_SMD:R_0805_2012Metric, F.Cu at (109.5, 35.5)
- added R8: R121,0805, Resistor_SMD:R_0805_2012Metric, F.Cu at (109.5, 38.5)
- added R9: R472,0805, Resistor_SMD:R_0805_2012Metric, F.Cu at (-52.2, 20.3)
- moved U6 91.2 mm to (-47.5, 20.3), turned to 90 degrees
- moved C7 67.5 mm to (-47.8, 26.5), turned to 180 degrees
- moved D3 48.9 mm to (-33.0, 43.2)
- moved U5 46.9 mm to (-55.1, 33.0)
- moved J3 37.2 mm to (-25.4, 40.6), turned to 180 degrees
Connections:
- U1 pad 18: unconnected-(U1-Pad18) -> +5V
- U1 pad 39: unconnected-(U1-Pad39) -> GND
- U3 pad 18: unconnected-(U3-Pad18) -> +5V
- U3 pad 39: unconnected-(U3-Pad39) -> GND
- U5 pad 18: unconnected-(U5-Pad18) -> +5V
- U5 pad 39: unconnected-(U5-Pad39) -> GND

Commit message: update,
Parts:
- added H1: MountingHole, footprint-lib:MountingHole_3.1mm_M3,rpi_like, F.Cu at (25.0, 115.0)
- added H2: MountingHole, footprint-lib:MountingHole_3.1mm_M3,rpi_like, F.Cu at (115.0, 115.0)
- added H3: MountingHole, footprint-lib:MountingHole_3.1mm_M3,rpi_like, F.Cu at (115.0, 25.0)
- added H4: MountingHole, footprint-lib:MountingHole_3.1mm_M3,rpi_like, F.Cu at (25.0, 25.0)
- added JP1: SolderJumper_2_Open_arrow, Jumper:SolderJumper-2_P1.3mm_Open_TrianglePad1.0x1.5mm, F.Cu at (98.1, 72.3)
- added JP2: SolderJumper_2_Open_arrow, Jumper:SolderJumper-2_P1.3mm_Open_TrianglePad1.0x1.5mm, F.Cu at (98.1, 74.9)
- added JP3: SolderJumper_2_Open_arrow, Jumper:SolderJumper-2_P1.3mm_Open_TrianglePad1.0x1.5mm, F.Cu at (98.1, 103.6)
- added JP4: SolderJumper_2_Open_arrow, Jumper:SolderJumper-2_P1.3mm_Open_TrianglePad1.0x1.5mm, F.Cu at (98.1, 106.1)
- added JP5: SolderJumper_2_Open_arrow, Jumper:SolderJumper-2_P1.3mm_Open_TrianglePad1.0x1.5mm, F.Cu at (94.6, 46.7)
- added JP6: SolderJumper_2_Open_arrow, Jumper:SolderJumper-2_P1.3mm_Open_TrianglePad1.0x1.5mm, F.Cu at (94.6, 49.2)
- moved R9 148.3 mm to (95.5, 33.5)
- moved U6 137.7 mm to (89.6, 33.7), turned to 0 degrees
- moved U5 132.3 mm to (77.1, 32.4), turned to -90 degrees
- moved C7 131.3 mm to (83.4, 33.5), turned to 90 degrees
- moved C8 127.2 mm to (88.1, 40.7)
- moved R10 127.2 mm to (90.6, 40.7)
- moved R12 118.6 mm to (87.8, 47.6), turned to -90 degrees
- moved D3 116.7 mm to (83.6, 47.7)
- moved J3 116.3 mm to (90.8, 46.7), turned to 0 degrees
- moved C9 115.4 mm to (83.0, 40.7)
- moved R11 115.4 mm to (85.6, 40.7)
- moved D2 82.7 mm to (84.1, 105.5)
- moved J2 71.1 mm to (94.3, 103.6)
- moved C6 69.6 mm to (88.6, 98.5), turned to 90 degrees
- moved C5 69.6 mm to (83.5, 98.5), turned to 90 degrees
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Connections:
- D2 pad 1: /stm32_1/CANH -> /stm32_2/CANH
- D2 pad 2: /stm32_1/CANL -> /stm32_2/CANL
- D3 pad 1: /stm32_1/CANH -> /stm32_3/CANH
- D3 pad 2: /stm32_1/CANL -> /stm32_3/CANL
- J2 pad 1: /stm32_1/CANH -> /stm32_2/CANH
- J2 pad 2: /stm32_1/CANL -> /stm32_2/CANL
- J3 pad 1: /stm32_1/CANH -> /stm32_3/CANH
- J3 pad 2: /stm32_1/CANL -> /stm32_3/CANL
- R10 pad 1: /stm32_1/CANL -> /stm32_3/CANL
- R11 pad 1: /stm32_1/CANH -> /stm32_3/CANH
- R12 pad 1: /stm32_1/CANH -> /stm32_3/CANH
- R12 pad 2: /stm32_1/CANL -> /stm32_3/CANL
- R6 pad 1: /stm32_1/CANL -> /stm32_2/CANL
- R7 pad 1: /stm32_1/CANH -> /stm32_2/CANH
- R8 pad 1: /stm32_1/CANH -> /stm32_2/CANH
- R8 pad 2: /stm32_1/CANL -> /stm32_2/CANL
- U4 pad 6: /stm32_1/CANL -> /stm32_2/CANL
- U4 pad 7: /stm32_1/CANH -> /stm32_2/CANH
- U6 pad 6: /stm32_1/CANL -> /stm32_3/CANL
- U6 pad 7: /stm32_1/CANH -> /stm32_3/CANH

Commit message: update,
Parts:
- JP1: renamed from JP6; footprint Jumper:SolderJumper-2_P1.3mm_Open_TrianglePad1.0x1.5mm -> Jumper:SolderJumper-2_P1.3mm_Open_RoundedPad1.0x1.5mm
- JP2: renamed from JP5; footprint Jumper:SolderJumper-2_P1.3mm_Open_TrianglePad1.0x1.5mm -> Jumper:SolderJumper-2_P1.3mm_Open_RoundedPad1.0x1.5mm
- JP3: renamed from JP1; footprint Jumper:SolderJumper-2_P1.3mm_Open_TrianglePad1.0x1.5mm -> Jumper:SolderJumper-2_P1.3mm_Open_RoundedPad1.0x1.5mm
- JP4: renamed from JP2; footprint Jumper:SolderJumper-2_P1.3mm_Open_TrianglePad1.0x1.5mm -> Jumper:SolderJumper-2_P1.3mm_Open_RoundedPad1.0x1.5mm
- JP5: renamed from JP4; footprint Jumper:SolderJumper-2_P1.3mm_Open_TrianglePad1.0x1.5mm -> Jumper:SolderJumper-2_P1.3mm_Open_RoundedPad1.0x1.5mm
- JP6: renamed from JP3; footprint Jumper:SolderJumper-2_P1.3mm_Open_TrianglePad1.0x1.5mm -> Jumper:SolderJumper-2_P1.3mm_Open_RoundedPad1.0x1.5mm
- moved R12 15.3 mm to (91.0, 105.0), turned to -90 degrees
- moved C9 12.7 mm to (94.0, 98.0)
- moved R9 12.5 mm to (96.0, 91.0)
- moved C7 7.55 mm to (84.0, 90.9)
- moved R10 7.12 mm to (84.0, 98.0), turned to -90 degrees
- moved R11 6.95 mm to (91.0, 98.0), turned to 90 degrees
- moved C8 1.63 mm to (87.0, 98.0)
- renumbered C7 to C1, C9 to C2, C8 to C3, C1 to C4, C2 to C5, C3 to C6, C5 to C7, C6 to C8, C4 to C9, D3 to D1, D1 to D2, D2 to D3, H4 to H1, H3 to H2, H1 to H3, H2 to H4, J3 to J1, J1 to J2, J2 to J3, R9 to R1, R7 to R10, R8 to R11, R5 to R12, R11 to R2, R12 to R3, R10 to R4, R1 to R5, R3 to R6, R2 to R7, R4 to R8, R6 to R9, U5 to U1, U6 to U2, U1 to U3, U2 to U4, U3 to U5, U4 to U6
Connections:
- C3 pad 1: Net-(C8-Pad1) (its old number) -> Net-(C3-Pad1)
- C5 pad 1: Net-(C2-Pad1) (its old number) -> Net-(C5-Pad1)
- C6 pad 1: Net-(C3-Pad1) -> Net-(C6-Pad1)
- C7 pad 1: Net-(C5-Pad1) -> +5V
- C9 pad 1: +5V -> Net-(C9-Pad1)
- D1 pad 1: /stm32_3/CANH -> /stm32_1/CANH
- D1 pad 2: /stm32_3/CANL -> /stm32_1/CANL
- D2 pad 1: /stm32_1/CANH -> /stm32_2/CANH
- D2 pad 2: /stm32_1/CANL -> /stm32_2/CANL
- D3 pad 1: /stm32_2/CANH -> /stm32_3/CANH
- D3 pad 2: /stm32_2/CANL -> /stm32_3/CANL
- J1 pad 1: /stm32_3/CANH -> /stm32_1/CANH
- J1 pad 2: /stm32_3/CANL -> /stm32_1/CANL
- J2 pad 1: /stm32_1/CANH -> /stm32_2/CANH
- J2 pad 2: /stm32_1/CANL -> /stm32_2/CANL
- J3 pad 1: /stm32_2/CANH -> /stm32_3/CANH
- J3 pad 2: /stm32_2/CANL -> /stm32_3/CANL
- JP1 pad 1: /stm32_3/CANL -> /stm32_1/CANH
- JP1 pad 2: /stm32_1/CAN_L -> /stm32_1/CAN_H
- JP2 pad 1: /stm32_3/CANH -> /stm32_1/CANL
- JP2 pad 2: /stm32_1/CAN_H -> /stm32_1/CAN_L
- JP3 pad 1: /stm32_1/CANH -> /stm32_2/CANH
- JP4 pad 1: /stm32_1/CANL -> /stm32_2/CANL
- JP5 pad 1: /stm32_2/CANL -> /stm32_3/CANH
- JP5 pad 2: /stm32_1/CAN_L -> /stm32_1/CAN_H
- JP6 pad 1: /stm32_2/CANH -> /stm32_3/CANL
- JP6 pad 2: /stm32_1/CAN_H -> /stm32_1/CAN_L
- R10 pad 1: /stm32_2/CANH -> /stm32_3/CANL
- R11 pad 1: /stm32_2/CANH -> /stm32_3/CANH
- R11 pad 2: /stm32_2/CANL -> Net-(C9-Pad1)
- R12 pad 1: GND -> /stm32_3/CANH
- R12 pad 2: Net-(R5-Pad2) (its old number) -> /stm32_3/CANL
- R2 pad 1: /stm32_3/CANH -> /stm32_1/CANL
- R3 pad 1: /stm32_3/CANH -> /stm32_1/CANH
- R3 pad 2: /stm32_3/CANL -> Net-(C3-Pad1)
- R4 pad 1: /stm32_3/CANL -> /stm32_1/CANH
- R4 pad 2: Net-(C8-Pad1) (its old number) -> /stm32_1/CANL
- R6 pad 1: /stm32_1/CANH -> /stm32_2/CANL
- R6 pad 2: Net-(C3-Pad1) -> Net-(C5-Pad1)
- R7 pad 1: /stm32_1/CANL -> /stm32_2/CANH
- R7 pad 2: Net-(C2-Pad1) (its old number) -> Net-(C6-Pad1)
- R8 pad 1: /stm32_1/CANH -> /stm32_2/CANH
- R8 pad 2: /stm32_1/CANL -> /stm32_2/CANL
- R9 pad 1: /stm32_2/CANL -> GND
- R9 pad 2: Net-(C5-Pad1) -> Net-(R9-Pad2)
- U1 pad 8: /stm32_3/CAN_RXD -> /stm32_1/CAN_RXD
- U1 pad 9: /stm32_3/CAN_TXD -> /stm32_1/CAN_TXD
- U2 pad 1: /stm32_3/CAN_TXD -> /stm32_1/CAN_TXD
- U2 pad 4: /stm32_3/CAN_RXD -> /stm32_1/CAN_RXD
- U2 pad 6: /stm32_3/CANL -> /stm32_1/CANL
- U2 pad 7: /stm32_3/CANH -> /stm32_1/CANH
- U3 pad 8: /stm32_1/CAN_RXD -> /stm32_2/CAN_RXD
- U3 pad 9: /stm32_1/CAN_TXD -> /stm32_2/CAN_TXD
- U4 pad 1: /stm32_1/CAN_TXD -> /stm32_2/CAN_TXD
- U4 pad 4: /stm32_1/CAN_RXD -> /stm32_2/CAN_RXD
- U4 pad 6: /stm32_1/CANL -> /stm32_2/CANL
- U4 pad 7: /stm32_1/CANH -> /stm32_2/CANH
- U5 pad 8: /stm32_2/CAN_RXD -> /stm32_3/CAN_RXD
- U5 pad 9: /stm32_2/CAN_TXD -> /stm32_3/CAN_TXD
- U6 pad 1: /stm32_2/CAN_TXD -> /stm32_3/CAN_TXD
- U6 pad 4: /stm32_2/CAN_RXD -> /stm32_3/CAN_RXD
- U6 pad 6: /stm32_2/CANL -> /stm32_3/CANL
- U6 pad 7: /stm32_2/CANH -> /stm32_3/CANH
- U6 pad 8: Net-(R5-Pad2) (its old number) -> Net-(R9-Pad2)
